File: pcb/usb-lcd.kicad_sch (KiCad schematic)
At the start: 12 parts, among them J1 USB, J2 Conn_01x02_Pin, U1 CH341A-EPP/MEM, Y1 12M

Commit message: Update PCB
Parts:
- removed C1: 15pF, Capacitor_SMD:C_0603_1608Metric, symbol Device:C
- removed C2: 15p, Capacitor_SMD:C_0603_1608Metric, symbol Device:C
- removed C3: 22u, Capacitor_SMD:C_0603_1608Metric, symbol Device:C
- removed R1: 2k2, Resistor_SMD:R_0603_1608Metric, symbol Device:R
- removed Y1: 12M, Crystal:Crystal_HC49-4H_Vertical, symbol Device:Crystal
- C4: footprint Capacitor_SMD:C_0603_1608Metric -> Capacitor_SMD:C_0805_2012Metric_Pad1.18x1.45mm_HandSolder; LCSC Part # (none) -> C519981
- C5: footprint Capacitor_SMD:C_0603_1608Metric -> Capacitor_SMD:C_0805_2012Metric_Pad1.18x1.45mm_HandSolder; LCSC Part # (none) -> C519911
- J1: LCSC Part # (none) -> C52016392
- J2: value Conn_01x02_Pin -> B/L; LCSC Part # (none) -> C52016390
- J3: renamed from DS1; value WC1602A -> LCD; LCSC Part # (none) -> C41375939
- RV1: LCSC Part # (none) -> C48997914
- U1: value CH341A-EPP/MEM -> CH341B-EPP/MEM; symbol CH341A:CH341A -> CH341A:CH341B-EPP/MEM; LCSC Part # C13517 -> C19185820
Connections:
- net GND: now also U1.13 (X1), U1.23 (SDA)
- no-connect marks 8 -> 9
Other:
- moved on the sheet: C4, C5, J1, J2, J3, RV1, U1
